Commit message: v0.2

File: arm_car_simulation/urdf/gazebo.urdf.xacro (robot description, xacro)
@@ -33,5 +33,5 @@
       </plugin>
     </gazebo>
-    <!-- <gazebo reference="${name}_footprint">
+    <gazebo reference="base_link">
       <gravity>true</gravity>
       <selfCollide>true</selfCollide>

File: arm_car_simulation/urdf/mobile_robot_body.urdf.xacro (robot description, xacro)
@@ -1,6 +1,6 @@
 <?xml version="1.0"?>
     <robot name="mobile_robot_body" xmlns:xacro="http://ros.org/wiki/xacro">
-      <property name="M_PI" value="3.14159"/>
-      <include filename="$(find arm_car_simulation)/urdf/gazebo.urdf.xacro"/>
+      <xacro:property name="M_PI" value="3.14159"/>
+      <xacro:include filename="$(find arm_car_simulation)/urdf/gazebo.urdf.xacro"/>
 <xacro:macro name="transmission_acro" params="joint_name">
 <transmission name="${joint_name}_tran1">
@@ -15,12 +15,12 @@
 </transmission>
 </xacro:macro>
-      <property name="base_x" value="0.33" />
-      <property name="base_y" value="0.33" />
+      <xacro:property name="base_x" value="0.33" />
+      <xacro:property name="base_y" value="0.33" />
       <xacro:macro name="mobile_robot_body">
         <link name="base_link">
         <inertial>
-          <origin xyz="0 0 0.055"/>
-          <mass value="1.0" />
-          <inertia ixx="1.0" ixy="0.0" ixz="0.0" iyy="1.0" iyz="0.0" izz="1.0"/>
+          <origin xyz="0 0 -0.1"/>
+          <mass value="150.0" />
+          <inertia ixx="10.0" ixy="0.0" ixz="0.0" iyy="10.0" iyz="0.0" izz="10.0"/>
         </inertial>
         <visual>
@@ -43,5 +43,5 @@
         <inertial>
           <origin  xyz="0.08 0.08 0.025"/>
-          <mass value="0.1" />
+          <mass value="1" />
            <inertia ixx="1.0" ixy="0.0" ixz="0.0" iyy="1.0" iyz="0.0" izz="1.0"/>
         </inertial>
@@ -65,5 +65,5 @@
         <parent link="base_link"/>
         <child link="left_front_wheel"/>
-        <origin rpy="0 1.57075 1.57075" xyz="0.3 0.3 0.1"/>
+        <origin rpy="0 1.57075 1.57075" xyz="0.3 0.325 0.1"/>
         <limit effort="100" velocity="100"/>
         <joint_properties damping="0.0" friction="0.0"/>
@@ -72,5 +72,5 @@
         <inertial>
           <origin xyz="0.08 -0.08 0.025"/>
-          <mass value="0.1" />
+          <mass value="1" />
            <inertia ixx="1.0" ixy="0.0" ixz="0.0" iyy="1.0" iyz="0.0" izz="1.0"/>
         </inertial>
@@ -94,5 +94,5 @@
         <parent link="base_link"/>
         <child link="right_front_wheel"/>
-        <origin rpy="0 1.57075 1.57075" xyz="0.3 -0.3 0.1"/>
+        <origin rpy="0 1.57075 1.57075" xyz="0.3 -0.325 0.1"/>
         <limit effort="100" velocity="100"/>
         <joint_properties damping="0.0" friction="0.0"/>
@@ -101,5 +101,5 @@
         <inertial>
           <origin xyz="-0.08 0.08 0.025"/>
-          <mass value="0.1" />
+          <mass value="1" />
            <inertia ixx="1.0" ixy="0.0" ixz="0.0" iyy="1.0" iyz="0.0" izz="1.0"/>
         </inertial>
@@ -123,5 +123,5 @@
         <parent link="base_link"/>
         <child link="left_back_wheel"/>
-        <origin rpy="0 1.57075 1.57075" xyz="-0.3 0.3 0.1"/>
+        <origin rpy="0 1.57075 1.57075" xyz="-0.3 0.325 0.1"/>
         <limit effort="100" velocity="100"/>
         <joint_properties damping="0.0" friction="0.0"/>
@@ -130,5 +130,5 @@
         <inertial>
            <origin xyz="-0.08 -0.08 0.025"/>
-           <mass value="0.1" />
+           <mass value="1" />
            <inertia ixx="1.0" ixy="0.0" ixz="0.0" iyy="1.0" iyz="0.0" izz="1.0"/>
         </inertial>
@@ -152,5 +152,5 @@
         <parent link="base_link"/>
         <child link="right_back_wheel"/>
-        <origin rpy="0 1.57075 1.57075" xyz="-0.3 -0.3 0.1"/>
+        <origin rpy="0 1.57075 1.57075" xyz="-0.3 -0.325 0.1"/>
         <limit effort="100" velocity="100"/>
         <joint_properties damping="0.0" friction="0.0"/>
@@ -180,7 +180,7 @@
         <parent link="base_link"/>
         <child link="head"/>
-        <origin xyz="0.2 0 0.38"/>
+        <origin xyz="0.1 0 0.38"/>
       </joint>
-    <xacro:transmission_acro joint_name="left_back_wheel_joint"/>
+  <xacro:transmission_acro joint_name="left_back_wheel_joint"/>
   <xacro:transmission_acro joint_name="right_back_wheel_joint"/>
   <xacro:transmission_acro joint_name="left_front_wheel_joint"/>

File: arm_car_simulation/urdf/ur3.urdf.xacro (robot description, xacro)
@@ -58,5 +58,5 @@
      wrist_2_lower_limit:=${-pi}    wrist_2_upper_limit:=${pi}
      wrist_3_lower_limit:=${-pi}    wrist_3_upper_limit:=${pi}">
-    <link name="${prefix}base_link" >
+    <link name="${prefix}ur_base_link" >
       <visual>
         <geometry>
@@ -77,5 +77,5 @@
     </link>
     <joint name="${prefix}shoulder_pan_joint" type="revolute">
-      <parent link="${prefix}base_link" />
+      <parent link="${prefix}ur_base_link" />
       <child link = "${prefix}shoulder_link" />
       <origin xyz="0.0 0.0 ${shoulder_height}" rpy="0.0 0.0 0.0" />

File: arm_car_simulation/urdf/ur5.urdf.xacro (robot description, xacro)
@@ -74,5 +74,5 @@
      wrist_2_lower_limit:=${-pi}    wrist_2_upper_limit:=${pi}
      wrist_3_lower_limit:=${-pi}    wrist_3_upper_limit:=${pi}">
-    <link name="${prefix}base_link" >
+    <link name="${prefix}ur_base_link" >
       <visual>
         <geometry>
@@ -93,5 +93,5 @@
     </link>
     <joint name="${prefix}shoulder_pan_joint" type="revolute">
-      <parent link="${prefix}base_link" />
+      <parent link="${prefix}ur_base_link" />
       <child link = "${prefix}shoulder_link" />
       <origin xyz="0.0 0.0 ${shoulder_height}" rpy="0.0 0.0 0.0" />
