Commit message: correct the error when the AGV rotates

File: ur_base_description/urdf/base/base.urdf.xacro (robot description, xacro)
@@ -61,11 +61,11 @@
         </collision>
       </link>
-      <joint name="left_front_wheel_joint" type="continuous">
+      <joint name="left_front_wheel_joint" type="fixed">
         <axis xyz="0 0 1"/>
         <parent link="base_link"/>
         <child link="left_front_wheel"/>
         <origin rpy="0 1.57075 1.57075" xyz="0.3 0.325 0.1"/>
-        <limit effort="100" velocity="100"/>
-        <joint_properties damping="0.0" friction="0.0"/>
+        <!-- <limit effort="100" velocity="100"/>
+        <joint_properties damping="0.0" friction="0.0"/>   -->
       </joint>
       <link name="right_front_wheel">
@@ -90,11 +90,11 @@
         </collision>
       </link>
-      <joint name="right_front_wheel_joint" type="continuous">
+      <joint name="right_front_wheel_joint" type="fixed">
         <axis xyz="0 0 1"/>
         <parent link="base_link"/>
         <child link="right_front_wheel"/>
         <origin rpy="0 1.57075 1.57075" xyz="0.3 -0.325 0.1"/>
-        <limit effort="100" velocity="100"/>
-        <joint_properties damping="0.0" friction="0.0"/>
+        <!-- <limit effort="100" velocity="100"/>
+        <joint_properties damping="0.0" friction="0.0"/>   -->
      </joint>
      <link name="left_back_wheel">
@@ -119,11 +119,11 @@
         </collision>
       </link>
-      <joint name="left_back_wheel_joint" type="continuous">
+      <joint name="left_back_wheel_joint" type="fixed">
         <axis xyz="0 0 1"/>
         <parent link="base_link"/>
         <child link="left_back_wheel"/>
         <origin rpy="0 1.57075 1.57075" xyz="-0.3 0.325 0.1"/>
-        <limit effort="100" velocity="100"/>
-        <joint_properties damping="0.0" friction="0.0"/>
+        <!-- <limit effort="100" velocity="100"/>
+        <joint_properties damping="0.0" friction="0.0"/>   -->
       </joint>
       <link name="right_back_wheel">
@@ -148,11 +148,11 @@
         </collision>
       </link>
-      <joint name="right_back_wheel_joint" type="continuous">
+      <joint name="right_back_wheel_joint" type="fixed">
         <axis xyz="0 0 1"/>
         <parent link="base_link"/>
         <child link="right_back_wheel"/>
         <origin rpy="0 1.57075 1.57075" xyz="-0.3 -0.325 0.1"/>
-        <limit effort="100" velocity="100"/>
-        <joint_properties damping="0.0" friction="0.0"/>
+        <!-- <limit effort="100" velocity="100"/>
+        <joint_properties damping="0.0" friction="0.0"/>   -->
       </joint>
       <link name="head">
@@ -182,8 +182,8 @@
         <origin xyz="0.1 0 0.38"/>
       </joint>
-  <xacro:transmission_acro joint_name="left_back_wheel_joint"/>
+  <!-- <xacro:transmission_acro joint_name="left_back_wheel_joint"/>
   <xacro:transmission_acro joint_name="right_back_wheel_joint"/>
   <xacro:transmission_acro joint_name="left_front_wheel_joint"/>
-  <xacro:transmission_acro joint_name="right_front_wheel_joint"/>
+  <xacro:transmission_acro joint_name="right_front_wheel_joint"/>  -->
       </xacro:macro>
 </robot>

File: ur_base_description/urdf/base/gazebo.urdf.xacro (robot description, xacro)
@@ -11,18 +11,30 @@
       <gazebo reference="right_front_wheel">
            <material>Gazebo/FlatBlack</material>
+            <gravity>true</gravity>
+           <selfCollide>true</selfCollide>
+           <kinematic>true</kinematic>
       </gazebo>
      <gazebo reference="right_back_wheel">
-           <material>Gazebo/FlatBlack</material>
+            <material>Gazebo/FlatBlack</material>
+            <gravity>true</gravity>
+           <selfCollide>true</selfCollide>
+           <kinematic>true</kinematic>
      </gazebo>
       <gazebo reference="left_front_wheel">
-            <material>Gazebo/FlatBlack</material>
+             <material>Gazebo/FlatBlack</material>
+            <gravity>true</gravity>
+           <selfCollide>true</selfCollide>
+           <kinematic>true</kinematic>
       </gazebo>
         <gazebo reference="left_back_wheel">
-            <material>Gazebo/FlatBlack</material>
+             <material>Gazebo/FlatBlack</material>
+            <gravity>true</gravity>
+           <selfCollide>true</selfCollide>
+           <kinematic>true</kinematic>
         </gazebo>
         <gazebo reference="head">
             <material>Gazebo/White</material>
         </gazebo>
-            <gazebo>
+   <gazebo>
       <plugin name="object_controller" filename="libgazebo_ros_planar_move.so">
         <commandTopic>cmd_vel</commandTopic>
@@ -36,5 +48,5 @@
       <gravity>true</gravity>
       <selfCollide>true</selfCollide>
-    </gazebo> -->
+    </gazebo>
    </xacro:macro>
 </robot>

File: ur_base_description/urdf/ur/ur10.urdf.xacro (robot description, xacro)
@@ -88,5 +88,5 @@
         <limit lower="${shoulder_pan_lower_limit}" upper="${shoulder_pan_upper_limit}" effort="330.0" velocity="2.16"/>
       </xacro:if>
-      <dynamics damping="0.0" friction="0.0"/>
+      <dynamics damping="0.0" friction="200.0"/>
     </joint>
     <link name="${prefix}shoulder_link">
